File: Directional_Coupler/Directional_Coupler.kicad_pcb (KiCad board)
At the start: 2 copper layers, 22 x 18 mm, 7 parts

Commit message: Minor slikscreen fixes and direction coupler prodcution files
Parts:
- H4: value Reverse -> Reflected
Other:
- board text added: "Fwd"
- board text added: "In"
- board text added: "JLCJLCJLCJLC"
- board text added: "Out"
- board text added: "Rfl"
Changed lines of the file:
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@@
 	(title_block
 		(title "Directional Coupler")
-		(date "2024-03-22")
+		(date "2024-05-05")
 		(rev "A0")
 		(company "TiZed")
@@
 			)
 		)
-		(property "Value" "Reverse"
-			(at 5.425 0.025 0)
+		(property "Value" "Reflected"
+			(at 6.1 0 0)
 			(unlocked yes)
 			(layer "F.Fab")
@@
 		(layer "Margin")
 	)
+	(gr_text "Rfl"
+		(at 107.75 57.7 0)
+		(layer "F.SilkS")
+		(effects
+			(font
+				(size 0.8 0.8)
+				(thickness 0.15)
+				(bold yes)
+			)
+			(justify left bottom)
+		)
+	)
+	(gr_text "JLCJLCJLCJLC"
+		(at 92.35 55.55 0)
+		(layer "F.SilkS")
+		(effects
+			(font
+				(size 0.8 0.8)
+				(thickness 0.15)
+			)
+			(justify left bottom)
+		)
+	)
+	(gr_text "Fwd"
+		(at 88.3 54.25 0)
+		(layer "F.SilkS")
+		(effects
+			(font
+				(size 0.8 0.8)
+				(thickness 0.15)
+				(bold yes)
+			)
+			(justify left bottom)
+		)
+	)
 	(gr_text "<"
 		(at 90 42 0)
@@
 			)
 			(justify left bottom)
+		)
+	)
+	(gr_text "Out"
+		(at 107.35 42.2 0)
+		(layer "F.SilkS")
+		(effects
+			(font
+				(size 0.8 0.8)
+				(thickness 0.15)
+				(bold yes)
+			)
+			(justify left bottom)
+		)
+	)
+	(gr_text "In"
+		(at 88.25 45.7 0)
+		(layer "F.SilkS")
+		(effects
+			(font
+				(size 0.8 0.8)
+				(thickness 0.15)
+				(bold yes)
+			)
+			(justify left bottom)
